Commit message: finish activity 6

File: src/rubot_mecanum_description/urdf/rubot.urdf (robot description, URDF)
Before this commit: robot rubot, 9 links, 8 joints
Joints:
- joint scan_joint: origin xyz=0 0 0.15 rpy=0 0 0 -> xyz=0 0 0.15 rpy=0 0 3.14

File: src/rubot_mecanum_description/urdf/rubot_custom.urdf (robot description, URDF)
Before this commit: robot rubot, 10 links, 9 joints
Links:
- removed link lidar_top_part
Joints:
- removed joint lidar_top_part_joint
- joint scan_joint: origin xyz=0 0 0.15 rpy=0 0 0 -> xyz=0 0 0.15 rpy=0 0 3.14
